Commit message: web ui nav update

File: description/gazebo_control.xacro (robot description, xacro)
@@ -7,5 +7,9 @@
             <right_joint>right_wheel_joint</right_joint>
             <wheel_separation>0.297</wheel_separation>
+<<<<<<< HEAD
             <wheel_diameter>0.066</wheel_diameter>
+=======
+            <wheel_diameter>0.106</wheel_diameter>
+>>>>>>> 51bf80f (web ui nav update)
             <!-- Limits -->
             <max_wheel_torque>200</max_wheel_torque>

File: description/lidar.xacro (robot description, xacro)
@@ -61,5 +61,9 @@
         <material>Gazebo/Black</material>
         <sensor name="laser" type="ray">
+<<<<<<< HEAD
             <pose> 0 0 0 0 0 3.14 </pose>
+=======
+            <pose>0 0 0 0 0 0</pose>
+>>>>>>> 51bf80f (web ui nav update)
             <visualize>true</visualize>
             <update_rate>10</update_rate>
@@ -89,5 +93,9 @@
         <material>Gazebo/Black</material>
         <sensor name="laser2" type="ray">
+<<<<<<< HEAD
             <pose> 0 0 0 0 0 3.14 </pose>
+=======
+            <pose>0 0 0 0 0 0</pose>
+>>>>>>> 51bf80f (web ui nav update)
             <visualize>true</visualize>
             <update_rate>10</update_rate>

File: description/robot_core.xacro (robot description, xacro)
@@ -89,5 +89,9 @@
         <parent link="base_link"/>
         <child link="left_wheel"/>
+<<<<<<< HEAD
         <origin xyz="0 ${wheel_offset_y} 0" rpy="-${pi/2} 0 0" />twist_mux
+=======
+        <origin xyz="0 ${wheel_offset_y} 0" rpy="-${pi/2} 0 0" />
+>>>>>>> 51bf80f (web ui nav update)
         <axis xyz="0 0 1"/>
     </joint>

File: description/ros2_control.xacro (robot description, xacro)
@@ -24,5 +24,8 @@
     <gazebo>
         <plugin name="gazebo_ros2_control" filename="libgazebo_ros2_control.so">
+<<<<<<< HEAD
             <parameters>$(find my_bot)/config/my_controllers.yaml</parameters>
+=======
+>>>>>>> 51bf80f (web ui nav update)
             <parameters>$(find my_bot)/config/gaz_ros2_ctl_use_sim.yaml</parameters>
         </plugin>

Commit message: Added Auto Relocation

File: description/gazebo_control.xacro (robot description, xacro)
@@ -7,9 +7,5 @@
             <right_joint>right_wheel_joint</right_joint>
             <wheel_separation>0.297</wheel_separation>
-<<<<<<< HEAD
-            <wheel_diameter>0.066</wheel_diameter>
-=======
             <wheel_diameter>0.106</wheel_diameter>
->>>>>>> 51bf80f (web ui nav update)
             <!-- Limits -->
             <max_wheel_torque>200</max_wheel_torque>

File: description/lidar.xacro (robot description, xacro)
@@ -61,9 +61,5 @@
         <material>Gazebo/Black</material>
         <sensor name="laser" type="ray">
-<<<<<<< HEAD
-            <pose> 0 0 0 0 0 3.14 </pose>
-=======
             <pose>0 0 0 0 0 0</pose>
->>>>>>> 51bf80f (web ui nav update)
             <visualize>true</visualize>
             <update_rate>10</update_rate>
@@ -93,9 +89,5 @@
         <material>Gazebo/Black</material>
         <sensor name="laser2" type="ray">
-<<<<<<< HEAD
-            <pose> 0 0 0 0 0 3.14 </pose>
-=======
             <pose>0 0 0 0 0 0</pose>
->>>>>>> 51bf80f (web ui nav update)
             <visualize>true</visualize>
             <update_rate>10</update_rate>

File: description/robot_core.xacro (robot description, xacro)
@@ -89,9 +89,5 @@
         <parent link="base_link"/>
         <child link="left_wheel"/>
-<<<<<<< HEAD
-        <origin xyz="0 ${wheel_offset_y} 0" rpy="-${pi/2} 0 0" />twist_mux
-=======
         <origin xyz="0 ${wheel_offset_y} 0" rpy="-${pi/2} 0 0" />
->>>>>>> 51bf80f (web ui nav update)
         <axis xyz="0 0 1"/>
     </joint>

File: description/ros2_control.xacro (robot description, xacro)
@@ -24,8 +24,4 @@
     <gazebo>
         <plugin name="gazebo_ros2_control" filename="libgazebo_ros2_control.so">
-<<<<<<< HEAD
-            <parameters>$(find my_bot)/config/my_controllers.yaml</parameters>
-=======
->>>>>>> 51bf80f (web ui nav update)
             <parameters>$(find my_bot)/config/gaz_ros2_ctl_use_sim.yaml</parameters>
         </plugin>
